Commit message: Fix the issue of motor shaking when dragging too fast.The reason for the jitter is zhe volocity limit in urdf!

File: swing_boy/urdf/swing_boy.urdf (robot description, URDF)
Before this commit: robot swing_boy, 6 links, 5 joints
Joints:
- joint joint1: limit lower=-3.14 upper=3.14 effort=3 velocity=1 -> lower=-3.14 upper=3.14 effort=3 velocity=5
- joint joint2: limit lower=-3.14 upper=3.14 effort=3 velocity=1 -> lower=-3.14 upper=3.14 effort=3 velocity=5
- joint joint3: limit lower=-3.14 upper=3.14 effort=3 velocity=1 -> lower=-3.14 upper=3.14 effort=3 velocity=5

Commit message: Fix arm hw.

File: swing_boy/urdf/swing_boy.urdf (robot description, URDF)
Before this commit: robot swing_boy, 6 links, 5 joints
Links:
- link link3: mass 0.058973 -> 0.108973
Joints:
- joint joint1: limit lower=-3.14 upper=3.14 effort=3 velocity=5 -> lower=-3.14 upper=3.14 effort=8 velocity=5
- joint joint2: limit lower=-3.14 upper=3.14 effort=3 velocity=5 -> lower=-3.14 upper=3.14 effort=8 velocity=5
- joint joint3: limit lower=-3.14 upper=3.14 effort=3 velocity=5 -> lower=-3.14 upper=3.14 effort=8 velocity=5
