Commit message: Right delta config.

File: delta/urdf/arm.transmission.xacro (robot description, xacro)
@@ -5,7 +5,8 @@
             <type>transmission_interface/SimpleTransmission</type>
             <actuator name="active_joint1_motor">
-                <mechanicalReduction>1</mechanicalReduction>
+                <mechanicalReduction>-1</mechanicalReduction>
             </actuator>
             <joint name="active_joint1">
+                <offset>0.437579</offset>
                 <hardwareInterface>hardware_interface/EffortJointInterface</hardwareInterface>
             </joint>
@@ -31,5 +32,5 @@
         <transmission name="trans_parallel_down_a_joint1">
             <type>transmission_interface/SimpleTransmission</type>
-            <actuator name="parallel_up_down_joint1_motor">
+            <actuator name="parallel_down_a_joint1_motor">
                 <mechanicalReduction>1</mechanicalReduction>
             </actuator>
@@ -50,7 +51,8 @@
             <type>transmission_interface/SimpleTransmission</type>
             <actuator name="active_joint2_motor">
-                <mechanicalReduction>1</mechanicalReduction>
+                <mechanicalReduction>-1</mechanicalReduction>
             </actuator>
             <joint name="active_joint2">
+                <offset>0.437579</offset>
                 <hardwareInterface>hardware_interface/EffortJointInterface</hardwareInterface>
             </joint>
@@ -76,5 +78,5 @@
         <transmission name="trans_parallel_down_a_joint2">
             <type>transmission_interface/SimpleTransmission</type>
-            <actuator name="parallel_up_down_joint2_motor">
+            <actuator name="parallel_down_a_joint2_motor">
                 <mechanicalReduction>1</mechanicalReduction>
             </actuator>
@@ -95,7 +97,8 @@
             <type>transmission_interface/SimpleTransmission</type>
             <actuator name="active_joint3_motor">
-                <mechanicalReduction>1</mechanicalReduction>
+                <mechanicalReduction>-1</mechanicalReduction>
             </actuator>
             <joint name="active_joint3">
+                <offset>0.437579</offset>
                 <hardwareInterface>hardware_interface/EffortJointInterface</hardwareInterface>
             </joint>
@@ -121,5 +124,5 @@
         <transmission name="trans_parallel_down_a_joint3">
             <type>transmission_interface/SimpleTransmission</type>
-            <actuator name="parallel_up_down_joint3_motor">
+            <actuator name="parallel_down_a_joint3_motor">
                 <mechanicalReduction>1</mechanicalReduction>
             </actuator>

File: delta/urdf/delta.urdf (robot description, URDF)
Before this commit: robot delta, 21 links, 20 joints
Joints:
- joint active_joint1: limit lower=-3.14 upper=3.14 effort=1 velocity=1 -> lower=-3.14 upper=3.14 effort=1 velocity=30
- joint active_joint2: limit lower=-3.14 upper=3.14 effort=1 velocity=1 -> lower=-3.14 upper=3.14 effort=1 velocity=30
- joint active_joint3: limit lower=-3.14 upper=3.14 effort=1 velocity=1 -> lower=-3.14 upper=3.14 effort=1 velocity=30

Commit message: New delta urdf and config.

File: delta/urdf/arm.transmission.xacro (robot description, xacro)
@@ -8,5 +8,5 @@
             </actuator>
             <joint name="active_joint1">
-                <offset>0.437579</offset>
+                <offset>-0.437579</offset>
                 <hardwareInterface>hardware_interface/EffortJointInterface</hardwareInterface>
             </joint>
@@ -54,5 +54,5 @@
             </actuator>
             <joint name="active_joint2">
-                <offset>0.437579</offset>
+                <offset>-0.437579</offset>
                 <hardwareInterface>hardware_interface/EffortJointInterface</hardwareInterface>
             </joint>
@@ -100,5 +100,5 @@
             </actuator>
             <joint name="active_joint3">
-                <offset>0.437579</offset>
+                <offset>-0.437579</offset>
                 <hardwareInterface>hardware_interface/EffortJointInterface</hardwareInterface>
             </joint>

File: delta/urdf/arm.urdf.xacro (robot description, xacro)
@@ -2,6 +2,6 @@
 <robot xmlns:xacro="http://www.ros.org/wiki/xacro" name="arm">
     <xacro:macro name="arm">
-        <xacro:property name="k_f" value="0.141067"/>
-        <xacro:property name="k_e" value="0.065287"/>
+        <xacro:property name="f" value="0.141067"/>
+        <xacro:property name="e" value="0.119853"/>
         <xacro:property name="r_f" value="0.09"/>
         <xacro:property name="r_e" value="0.192"/>
@@ -360,5 +360,5 @@
             <parent link="base_link"/>
             <child link="active_arm_2"/>
-            <origin xyz="-${(active_joint_d)*cos(pi/6)} ${(active_joint_d)*sin(pi/6)} 0." rpy="0 0 ${v120_deg_2_rad}"/>
+            <origin xyz="${(active_joint_d)*cos(pi/6)} ${(active_joint_d)*sin(pi/6)} 0." rpy="0 0 ${v120_deg_2_rad}"/>
             <axis xyz="1 0 0"/>
             <limit lower="-3.14" upper="3.14" velocity="1" effort="1"/>
@@ -501,5 +501,5 @@
             <parent link="base_link"/>
             <child link="active_arm_3"/>
-            <origin xyz="${(active_joint_d)*cos(pi/6)} ${(active_joint_d)*sin(pi/6)} 0." rpy="0 0 -${v120_deg_2_rad}"/>
+            <origin xyz="-${(active_joint_d)*cos(pi/6)} ${(active_joint_d)*sin(pi/6)} 0." rpy="0 0 -${v120_deg_2_rad}"/>
             <axis xyz="1 0 0"/>
             <limit lower="-3.14" upper="3.14" velocity="1" effort="1"/>

File: delta/urdf/delta.urdf (robot description, URDF)
Before this commit: robot delta, 21 links, 20 joints
Joints:
- joint active_joint1: limit lower=-3.14 upper=3.14 effort=1 velocity=30 -> lower=-3.14 upper=3.14 effort=1 velocity=1
- joint active_joint2: limit lower=-3.14 upper=3.14 effort=1 velocity=30 -> lower=-3.14 upper=3.14 effort=1 velocity=1; origin xyz=-0.03526542046750613 0.020360499999999997 0. rpy=0 0 -2.09439504 -> xyz=0.03526542046750613 0.020360499999999997 0. rpy=0 0 2.09439504
- joint active_joint3: limit lower=-3.14 upper=3.14 effort=1 velocity=30 -> lower=-3.14 upper=3.14 effort=1 velocity=1; origin xyz=0.03526542046750613 0.020360499999999997 0. rpy=0 0 2.09439504 -> xyz=-0.03526542046750613 0.020360499999999997 0. rpy=0 0 -2.09439504
